Commit message: gripper added to keyboard application

File: open_manipulator_pro_description/urdf/open_manipulator_pro_with_gripper.gazebo.xacro (robot description, xacro)
@@ -47,18 +47,18 @@
     <material>Gazebo/Grey</material>
   </gazebo>
-  <!-- grip main link -->
-  <gazebo reference="grip_main_link">
+  <!-- gripper main link -->
+  <gazebo reference="gripper_main_link">
     <mu1>0.2</mu1>
     <mu2>0.2</mu2>
     <material>Gazebo/Grey</material>
   </gazebo>
-  <!-- grip link -->
-  <gazebo reference="grip_link">
+  <!-- gripper link -->
+  <gazebo reference="gripper_link">
     <mu1>0.2</mu1>
     <mu2>0.2</mu2>
     <material>Gazebo/Grey</material>
   </gazebo>
-  <!-- grip 1 link -->
-  <gazebo reference="grip_1_link">
+  <!-- gripper 1 link -->
+  <gazebo reference="gripper_sub_link">
     <mu1>0.2</mu1>
     <mu2>0.2</mu2>

File: open_manipulator_pro_description/urdf/open_manipulator_pro_with_gripper.urdf.xacro (robot description, xacro)
@@ -227,5 +227,5 @@
   <joint name="joint6" type="revolute">
     <parent link="link6"/>
-    <child link="grip_main_link"/>
+    <child link="gripper_main_link"/>
     <origin xyz="0.12300 -0.04500 0.00000" rpy="0 0 0"/>
     <axis xyz="1 0 0"/>
@@ -236,15 +236,15 @@
   <xacro:SimpleTransmission n="6" joint="joint6" />
   <!-- gripper main link -->
-  <link name="grip_main_link">
-    <collision>
-      <origin xyz="0 0 0" rpy="0 0 0" />
-      <geometry>
-        <mesh filename="package://open_manipulator_pro_description/meshes/grip_main_link.stl" scale="0.001 0.001 0.001"/>
-      </geometry>
-    </collision>
-    <visual>
-      <origin xyz="0 0 0" rpy="0 0 0" />
-      <geometry>
-        <mesh filename="package://open_manipulator_pro_description/meshes/grip_main_link.stl" scale="0.001 0.001 0.001"/>
+  <link name="gripper_main_link">
+    <collision>
+      <origin xyz="0 0 0" rpy="0 0 0" />
+      <geometry>
+        <mesh filename="package://open_manipulator_pro_description/meshes/gripper_main_link.stl" scale="0.001 0.001 0.001"/>
+      </geometry>
+    </collision>
+    <visual>
+      <origin xyz="0 0 0" rpy="0 0 0" />
+      <geometry>
+        <mesh filename="package://open_manipulator_pro_description/meshes/gripper_main_link.stl" scale="0.001 0.001 0.001"/>
       </geometry>
       <material name="grey"/>
@@ -257,28 +257,28 @@
   </link>
   <!-- gripper joint -->
-  <joint name="grip" type="revolute">
+  <joint name="gripper" type="revolute">
     <axis xyz="0 0 1" />
-    <!-- <origin xyz="0.0552 -0.0133 0" rpy="0 0 0"/> -->
-    <origin xyz="0.0552 -0.0370 0" rpy="0 0 ${4.0*pi/18.0}"/>
-    <parent link="grip_main_link"/>
-    <child link="grip_link"/>
+    <!-- <origin xyz="0.0552 -0.0370 0" rpy="0 0 ${4.0*pi/18.0}"/> -->
+    <origin xyz="0.0552 -0.0370 0" rpy="0 0 0"/>
+    <parent link="gripper_main_link"/>
+    <child link="gripper_link"/>
     <limit velocity="6.5" effort="1000" lower="0.0" upper="${65.0*pi/180.0}" />
     <dynamics damping="0.1" friction="0.0" />
   </joint>
-  <!-- Transmission grip -->
-  <xacro:SimpleTransmission n="_grip" joint="grip" />
+  <!-- Transmission gripper -->
+  <xacro:SimpleTransmission n="_gripper" joint="gripper" />
   <!-- gripper link -->
-  <link name="grip_link">
-    <collision>
-      <origin xyz="0 0 0" rpy="0 0 0" />
-      <geometry>
-        <mesh filename="package://open_manipulator_pro_description/meshes/grip_link.stl" scale="0.001 0.001 0.001"/>
-      </geometry>
-      <material name="grey"/>
-    </collision>
-    <visual>
-      <origin xyz="0 0 0" rpy="0 0 0" />
-      <geometry>
-        <mesh filename="package://open_manipulator_pro_description/meshes/grip_link.stl" scale="0.001 0.001 0.001"/>
+  <link name="gripper_link">
+    <collision>
+      <origin xyz="0 0 0" rpy="0 0 0" />
+      <geometry>
+        <mesh filename="package://open_manipulator_pro_description/meshes/gripper_link.stl" scale="0.001 0.001 0.001"/>
+      </geometry>
+      <material name="grey"/>
+    </collision>
+    <visual>
+      <origin xyz="0 0 0" rpy="0 0 0" />
+      <geometry>
+        <mesh filename="package://open_manipulator_pro_description/meshes/gripper_link.stl" scale="0.001 0.001 0.001"/>
       </geometry>
       <material name="grey"/>
@@ -291,28 +291,28 @@
   </link>
   <!-- gripper joint 1 -->
-  <joint name="grip_1" type="revolute">
+  <joint name="gripper_sub" type="revolute">
     <axis xyz="0 0 -1" />
-    <!-- <origin xyz="0.0552 0.0133 0" rpy="0 0 0"/> -->
-    <origin xyz="0.0552 0.0370 0" rpy="0 0 ${-4.0*pi/18.0}"/>
-    <parent link="grip_main_link"/>
-    <child link="grip_1_link"/>
+    <!-- <origin xyz="0.0552 0.0370 0" rpy="0 0 ${-4.0*pi/18.0}"/> -->
+    <origin xyz="0.0552 0.0370 0" rpy="0 0 0"/>
+    <parent link="gripper_main_link"/>
+    <child link="gripper_sub_link"/>
     <limit velocity="6.5" effort="1000" lower="0.0" upper="${65.0*pi/180.0}" />
     <dynamics damping="0.1" friction="0.0" />
   </joint>
-  <!-- Transmission grip -->
-  <xacro:SimpleTransmission n="_grip_1" joint="grip_1" />
+  <!-- Transmission gripper -->
+  <xacro:SimpleTransmission n="_gripper_sub" joint="gripper_sub" />
   <!-- gripper 1 link -->
-  <link name="grip_1_link">
-    <collision>
-      <origin xyz="0 0 0" rpy="0 0 0" />
-      <geometry>
-        <mesh filename="package://open_manipulator_pro_description/meshes/grip_1_link.stl" scale="0.001 0.001 0.001"/>
-      </geometry>
-      <material name="grey"/>
-    </collision>
-    <visual>
-      <origin xyz="0 0 0" rpy="0 0 0" />
-      <geometry>
-        <mesh filename="package://open_manipulator_pro_description/meshes/grip_1_link.stl" scale="0.001 0.001 0.001"/>
+  <link name="gripper_sub_link">
+    <collision>
+      <origin xyz="0 0 0" rpy="0 0 0" />
+      <geometry>
+        <mesh filename="package://open_manipulator_pro_description/meshes/gripper_sub_link.stl" scale="0.001 0.001 0.001"/>
+      </geometry>
+      <material name="grey"/>
+    </collision>
+    <visual>
+      <origin xyz="0 0 0" rpy="0 0 0" />
+      <geometry>
+        <mesh filename="package://open_manipulator_pro_description/meshes/gripper_sub_link.stl" scale="0.001 0.001 0.001"/>
       </geometry>
       <material name="grey"/>
@@ -325,6 +325,6 @@
   </link>
   <!-- gripper main fixed joint-->
-  <joint name="grip_main_fixed" type="fixed">
-    <parent link="grip_main_link"/>
+  <joint name="gripper_main_fixed" type="fixed">
+    <parent link="gripper_main_link"/>
     <child link="end_effector"/>
     <origin xyz="0.14 0.0 0.0" rpy="0 0 0" />
