Commit message: minor change in package.xml

File: open_manipulator_pro_description/urdf/open_manipulator_pro_with_gripper.urdf.xacro (robot description, xacro)
@@ -341,9 +341,5 @@
       <origin xyz="0.0 0.0 0.0" rpy="0 0 0" />
       <mass value="0.001" />
-      <inertia
-	  ixx="1.0" ixy="0.0" ixz="0.0"
-	  iyy="1.0" iyz="0.0"
-	  izz="1.0"/>
-    </inertial>
+      <inertia ixx="1.0" ixy="0.0" ixz="0.0" iyy="1.0" iyz="0.0" izz="1.0" />
   </link>
 </robot>

Commit message: gripper added to controller, om-lib

File: open_manipulator_pro_description/urdf/open_manipulator_pro_with_gripper.urdf.xacro (robot description, xacro)
@@ -7,7 +7,7 @@
   <xacro:property name="pi" value="3.141592654" />
   <!-- Import all Gazebo-customization elements, including Gazebo colors -->
-  <xacro:include filename="$(find manipulator_h_description)/urdf/open_manipulator_pro_with_gripper.gazebo" />
+  <xacro:include filename="$(find open_manipulator_pro_description)/urdf/open_manipulator_pro_with_gripper.gazebo" />
   <!-- Import Rviz colors -->
-  <xacro:include filename="$(find manipulator_h_description)/urdf/materials.xacro" />
+  <xacro:include filename="$(find open_manipulator_pro_description)/urdf/materials.xacro" />
   <!-- Transmission macro -->
   <xacro:macro name="SimpleTransmission" params="joint n">
@@ -49,5 +49,4 @@
     <inertial>
       <origin xyz="0.00023 0.00000 0.06223" rpy="0 0 0"/>
-      <!--<origin xyz="0.00023 0.00000 -0.06377" rpy="0 0 0"/>-->
       <mass value="0.85644"/>
       <inertia ixx="1.0" ixy="0.0" ixz="0.0" iyy="1.0" iyz="0.0" izz="1.0" />
@@ -342,4 +341,5 @@
       <mass value="0.001" />
       <inertia ixx="1.0" ixy="0.0" ixz="0.0" iyy="1.0" iyz="0.0" izz="1.0" />
+    </inertial>
   </link>
 </robot>

Commit message: gripper added to controller, moveit

File: open_manipulator_pro_description/urdf/open_manipulator_pro_with_gripper.urdf.xacro (robot description, xacro)
@@ -259,5 +259,6 @@
   <joint name="grip" type="revolute">
     <axis xyz="0 0 1" />
-    <origin xyz="0.0552 -0.0133 0" rpy="0 0 ${-4.0*pi/18.0}"/>
+    <!-- <origin xyz="0.0552 -0.0133 0" rpy="0 0 0"/> -->
+    <origin xyz="0.0552 -0.0370 0" rpy="0 0 ${4.0*pi/18.0}"/>
     <parent link="grip_main_link"/>
     <child link="grip_link"/>
@@ -292,5 +293,6 @@
   <joint name="grip_1" type="revolute">
     <axis xyz="0 0 -1" />
-    <origin xyz="0.0552 0.0133 0" rpy="0 0 ${4.0*pi/18.0}"/>
+    <!-- <origin xyz="0.0552 0.0133 0" rpy="0 0 0"/> -->
+    <origin xyz="0.0552 0.0370 0" rpy="0 0 ${-4.0*pi/18.0}"/>
     <parent link="grip_main_link"/>
     <child link="grip_1_link"/>
@@ -326,5 +328,5 @@
     <parent link="grip_main_link"/>
     <child link="end_effector"/>
-    <origin xyz="0.12 0.0 0.0" rpy="0 0 0" />
+    <origin xyz="0.14 0.0 0.0" rpy="0 0 0" />
   </joint>
   <!-- End Effector -->

Commit message: changed m->rad for gripper, set gripper init pos

File: open_manipulator_pro_description/urdf/open_manipulator_pro_with_gripper.urdf.xacro (robot description, xacro)
@@ -258,10 +258,10 @@
   <!-- gripper joint -->
   <joint name="gripper" type="revolute">
-    <axis xyz="0 0 1" />
-    <!-- <origin xyz="0.0552 -0.0370 0" rpy="0 0 ${4.0*pi/18.0}"/> -->
-    <origin xyz="0.0552 -0.0370 0" rpy="0 0 0"/>
+    <axis xyz="0 0 -1" />
+    <origin xyz="0.0552 -0.0460 0" rpy="0 0 ${45.0*pi/180.0}"/>
+    <!-- <origin xyz="0.0552 -0.0370 0" rpy="0 0 0"/> -->
     <parent link="gripper_main_link"/>
     <child link="gripper_link"/>
-    <limit velocity="6.5" effort="1000" lower="0.0" upper="${65.0*pi/180.0}" />
+    <limit velocity="6.5" effort="1000" lower="0.0" upper="${740.0/2048.0*pi}" />
     <dynamics damping="0.1" friction="0.0" />
   </joint>
@@ -292,10 +292,10 @@
   <!-- gripper joint 1 -->
   <joint name="gripper_sub" type="revolute">
-    <axis xyz="0 0 -1" />
-    <!-- <origin xyz="0.0552 0.0370 0" rpy="0 0 ${-4.0*pi/18.0}"/> -->
-    <origin xyz="0.0552 0.0370 0" rpy="0 0 0"/>
+    <axis xyz="0 0 1" />
+    <origin xyz="0.0552 0.0460 0" rpy="0 0 ${-45.0*pi/180.0}"/>
+    <!-- <origin xyz="0.0552 0.0370 0" rpy="0 0 0"/> -->
     <parent link="gripper_main_link"/>
     <child link="gripper_sub_link"/>
-    <limit velocity="6.5" effort="1000" lower="0.0" upper="${65.0*pi/180.0}" />
+    <limit velocity="6.5" effort="1000" lower="0.0" upper="${740.0/2048.0*pi}" />
     <dynamics damping="0.1" friction="0.0" />
   </joint>
