Commit message: urdf axes modified

File: open_manipulator_pro_description/urdf/open_manipulator_pro.urdf.xacro (robot description, xacro)
@@ -49,5 +49,4 @@
     <inertial>
       <origin xyz="0.00023 0.00000 0.06223" rpy="0 0 0"/>
-      <!--<origin xyz="0.00023 0.00000 -0.06377" rpy="0 0 0"/>-->
       <mass value="0.85644"/>
       <inertia ixx="1.0" ixy="0.0" ixz="0.0" iyy="1.0" iyz="0.0" izz="1.0" />
@@ -93,5 +92,5 @@
     <parent link="link2"/>
     <child link="link3"/>
-    <origin xyz="0.0 0.069 0.033" rpy="0 0 0"/>
+    <origin xyz="0.0 0.0 0.033" rpy="0 0 0"/>
     <axis xyz="0 1 0"/>
     <limit velocity="6.5" effort="1000" lower="${-pi*0.5}" upper="${pi*0.5}" />
@@ -103,5 +102,5 @@
   <link name="link3">
     <collision>
-      <origin xyz="0 0 0" rpy="0 0 0"/>
+      <origin xyz="0 0.069 0" rpy="0 0 0"/>
       <geometry>
         <mesh filename="package://open_manipulator_pro_description/meshes/link_3.stl" scale="0.001 0.001 0.001"/>
@@ -109,5 +108,5 @@
     </collision>
     <visual>
-      <origin xyz="0 0 0" rpy="0 0 0"/>
+      <origin xyz="0 0.069 0" rpy="0 0 0"/>
       <geometry>
         <mesh filename="package://open_manipulator_pro_description/meshes/link_3.stl" scale="0.001 0.001 0.001"/>
@@ -116,6 +115,5 @@
     </visual>
     <inertial>
-      <origin xyz="0.01768 -0.06881 0.20524" rpy="0 0 0"/>
-      <!--<origin xyz="-0.01232 -0.05731 -0.05876" rpy="0 0 0"/>-->
+      <origin xyz="0.01768 0.00019 0.20524" rpy="0 0 0"/>
       <mass value="1.30260"/>
       <inertia ixx="1.0" ixy="0.0" ixz="0.0" iyy="1.0" iyz="0.0" izz="1.0" />
@@ -127,5 +125,5 @@
     <parent link="link3"/>
     <child link="link4"/>
-    <origin xyz="0.03000 -0.01150 0.26400" rpy="0 0 0"/>
+    <origin xyz="0.03000 0.0 0.26400" rpy="0 0 0"/>
     <axis xyz="0 1 0"/>
     <limit velocity="6.5" effort="1000" lower="${-pi*0.5}" upper="${pi*0.5}" />
@@ -137,5 +135,5 @@
   <link name="link4">
     <collision>
-      <origin xyz="0 0 0" rpy="0 0 0"/>
+      <origin xyz="0 0.05750 0" rpy="0 0 0"/>
       <geometry>
         <mesh filename="package://open_manipulator_pro_description/meshes/link_4.stl" scale="0.001 0.001 0.001"/>
@@ -143,5 +141,5 @@
     </collision>
     <visual>
-      <origin xyz="0 0 0" rpy="0 0 0"/>
+      <origin xyz="0 0.05750 0" rpy="0 0 0"/>
       <geometry>
         <mesh filename="package://open_manipulator_pro_description/meshes/link_4.stl" scale="0.001 0.001 0.001"/>
@@ -150,6 +148,5 @@
     </visual>
     <inertial>
-      <origin xyz="0.12475 -0.05716 0.02979" rpy="0 0 0"/>
-      <!--<origin xyz="-0.07025 0.00034 -0.00021" rpy="0 0 0"/>-->
+      <origin xyz="-0.07025 0.00034 -0.00021" rpy="0 0 0"/>
       <mass value="1.15977"/>
       <inertia ixx="1.0" ixy="0.0" ixz="0.0" iyy="1.0" iyz="0.0" izz="1.0" />
@@ -161,5 +158,5 @@
     <parent link="link4"/>
     <child link="link5"/>
-    <origin xyz="0.19500 -0.05750 0.03000" rpy="0 0 0"/>
+    <origin xyz="0.19500 0.0 0.03000" rpy="0 0 0"/>
     <axis xyz="1 0 0"/>
     <limit velocity="6.5" effort="1000" lower="${-pi*0.5}" upper="${pi*0.5}" />
@@ -195,5 +192,5 @@
     <parent link="link5"/>
     <child link="link6"/>
-    <origin xyz="0.06300 0.04500 0.00000" rpy="0 0 0"/>
+    <origin xyz="0.06300 0.00 0.00000" rpy="0 0 0"/>
     <axis xyz="0 1 0"/>
     <limit velocity="6.5" effort="1000" lower="${-pi*0.5}" upper="${pi*0.5}" />
@@ -205,5 +202,5 @@
   <link name="link6">
     <collision>
-      <origin xyz="0 0 0" rpy="0 0 0"/>
+      <origin xyz="0 0.04500 0" rpy="0 0 0"/>
       <geometry>
         <mesh filename="package://open_manipulator_pro_description/meshes/link_6.stl" scale="0.001 0.001 0.001"/>
@@ -211,5 +208,5 @@
     </collision>
     <visual>
-      <origin xyz="0 0 0" rpy="0 0 0"/>
+      <origin xyz="0 0.04500 0" rpy="0 0 0"/>
       <geometry>
         <mesh filename="package://open_manipulator_pro_description/meshes/link_6.stl" scale="0.001 0.001 0.001"/>
@@ -218,6 +215,6 @@
     </visual>
     <inertial>
-      <origin xyz="0.06831 -0.04457 0.00000" rpy="0 0 0"/>
-      <!--<origin xyz="-0.05469 0.00043 0.00000" rpy="0 0 0"/>-->
+      <!-- <origin xyz="0.06831 -0.04457 0.00000" rpy="0 0 0"/> -->
+      <origin xyz="-0.05469 0.00043 0.00000" rpy="0 0 0"/>
       <mass value="0.43273"/>
       <inertia ixx="1.0" ixy="0.0" ixz="0.0" iyy="1.0" iyz="0.0" izz="1.0" />
@@ -229,5 +226,5 @@
     <parent link="link6"/>
     <child link="end_link"/>
-    <origin xyz="0.12300 -0.04500 0.00000" rpy="0 0 0"/>
+    <origin xyz="0.12300 0.000 0.00000" rpy="0 0 0"/>
     <axis xyz="1 0 0"/>
     <limit velocity="6.5" effort="1000" lower="${-pi*0.5}" upper="${pi*0.5}" />

Commit message: control gui joint state display bug fixed

File: open_manipulator_pro_description/urdf/open_manipulator_pro.urdf.xacro (robot description, xacro)
@@ -2,6 +2,4 @@
 <!-- Revolute-Revolute Manipulator -->
 <robot name="open_manipulator_pro" xmlns:xacro="http://www.ros.org/wiki/xacro">
-  <!-- some parameters -->
-  <xacro:property name="pi" value="3.141592654" />
   <!-- some parameters -->
   <xacro:property name="pi" value="3.141592654" />
