Commit message: ROS2 initial upload

File: open_manipulator_pro_description/urdf/materials.xacro (robot description, xacro)
@@ -3,4 +3,10 @@
   <material name="black">
     <color rgba="0.0 0.0 0.0 1.0"/>
+  </material>
+  <material name="white">
+    <color rgba="1.0 1.0 1.0 1.0"/>
+  </material>
+  <material name="red">
+    <color rgba="0.8 0.0 0.0 1.0"/>
   </material>
   <material name="blue">
@@ -19,9 +25,3 @@
     <color rgba="${222/255} ${207/255} ${195/255} 1.0"/>
   </material>
-  <material name="red">
-    <color rgba="0.8 0.0 0.0 1.0"/>
-  </material>
-  <material name="white">
-    <color rgba="1.0 1.0 1.0 1.0"/>
-  </material>
 </robot>

File: open_manipulator_pro_description/urdf/open_manipulator_pro.gazebo.xacro (robot description, xacro)
@@ -1,55 +1,40 @@
 <?xml version="1.0"?>
-<robot>
+<robot xmlns:xacro="http://ros.org/wiki/xacro">
+  <!-- Gazebo Reference macro -->
+  <xacro:macro name="RefLink" params="ref">
+    <gazebo reference="${ref}">
+      <kp>1000000.0</kp>
+      <kd>100.0</kd>
+      <mu1>30.0</mu1>
+      <mu2>30.0</mu2>
+      <maxVel>1.0</maxVel>
+      <minDepth>0.001</minDepth>
+      <material>Gazebo/DarkGrey</material>
+    </gazebo>
+  </xacro:macro>
+  <!-- World -->
+  <gazebo reference="world">
+  </gazebo>
+  <!-- Link1 -->
+  <RefLink ref="link1"/>
+  <!-- Link2 -->
+  <RefLink ref="link2"/>
+  <!-- Link3 -->
+  <RefLink ref="link3"/>
+  <!-- Link4 -->
+  <RefLink ref="link4"/>
+  <!-- Link5 -->
+  <RefLink ref="link5"/>
+  <!-- gripper_link -->
+  <RefLink ref="link6"/>
+  <!-- gripper_link_sub -->
+  <RefLink ref="end_link"/>
   <!-- ros_control plugin -->
   <gazebo>
     <plugin name="gazebo_ros_control" filename="libgazebo_ros_control.so">
       <robotNamespace>open_manipulator_pro</robotNamespace>
+      <controlPeriod>0.001</controlPeriod>
       <robotSimType>gazebo_ros_control/DefaultRobotHWSim</robotSimType>
     </plugin>
   </gazebo>
-  <!-- World -->
-  <gazebo reference="world">
-  </gazebo>
-  <!-- Link1 -->
-  <gazebo reference="link1">
-    <mu1>0.2</mu1>
-    <mu2>0.2</mu2>
-    <material>Gazebo/Grey</material>
-  </gazebo>
-  <!-- Link2 -->
-  <gazebo reference="link2">
-    <mu1>0.2</mu1>
-    <mu2>0.2</mu2>
-    <material>Gazebo/Grey</material>
-  </gazebo>
-  <!-- Link3 -->
-  <gazebo reference="link3">
-    <mu1>0.2</mu1>
-    <mu2>0.2</mu2>
-    <material>Gazebo/Grey</material>
-  </gazebo>
-  <!-- Link4 -->
-  <gazebo reference="link4">
-    <mu1>0.2</mu1>
-    <mu2>0.2</mu2>
-    <material>Gazebo/Grey</material>
-  </gazebo>
-  <!-- Link5 -->
-  <gazebo reference="link5">
-    <mu1>0.2</mu1>
-    <mu2>0.2</mu2>
-    <material>Gazebo/Grey</material>
-  </gazebo>
-  <!-- Link6 -->
-  <gazebo reference="link6">
-    <mu1>0.2</mu1>
-    <mu2>0.2</mu2>
-    <material>Gazebo/Grey</material>
-  </gazebo>
-  <!-- End Link -->
-  <gazebo reference="end_link">
-    <mu1>0.2</mu1>
-    <mu2>0.2</mu2>
-    <material>Gazebo/Grey</material>
-  </gazebo>
 </robot>

File: open_manipulator_pro_description/urdf/open_manipulator_pro.urdf.xacro (robot description, xacro)
@@ -1,13 +1,42 @@
 <?xml version="1.0"?>
-<!-- Revolute-Revolute Manipulator -->
-<robot name="open_manipulator_pro" xmlns:xacro="http://www.ros.org/wiki/xacro">
+<!-- OpenManipulator Chain -->
+<robot name="open_manipulator_pro" xmlns:xacro="http://ros.org/wiki/xacro">
   <!-- some parameters -->
-  <xacro:property name="pi" value="3.141592654" />
-  <!-- some parameters -->
-  <xacro:property name="pi" value="3.141592654" />
+  <!-- <xacro:property name="pi" value="3.141592654" /> -->
   <!-- Import all Gazebo-customization elements, including Gazebo colors -->
   <xacro:include filename="$(find open_manipulator_pro_description)/urdf/open_manipulator_pro.gazebo.xacro" />
   <!-- Import Rviz colors -->
-  <xacro:include filename="$(find open_manipulator_pro_description)/urdf/materials.xacro" />
+  <!-- <xacro:include filename="$(find open_manipulator_pro_description)/urdf/materials.xacro" /> -->
+  <!-- Init colour -->
+  <material name="black">
+      <color rgba="0.0 0.0 0.0 1.0"/>
+  </material>
+  <material name="dark">
+    <color rgba="0.3 0.3 0.3 1.0"/>
+  </material>
+  <material name="light_black">
+    <color rgba="0.4 0.4 0.4 1.0"/>
+  </material>
+  <material name="blue">
+    <color rgba="0.0 0.0 0.8 1.0"/>
+  </material>
+  <material name="green">
+    <color rgba="0.0 0.8 0.0 1.0"/>
+  </material>
+  <material name="grey">
+    <color rgba="0.5 0.5 0.5 1.0"/>
+  </material>
+  <material name="orange">
+    <color rgba="1.0 0.4235 0.0392 1.0"/>
+  </material>
+  <material name="brown">
+    <color rgba="0.8706 0.8118 0.7647 1.0"/>
+  </material>
+  <material name="red">
+    <color rgba="0.8 0.0 0.0 1.0"/>
+  </material>
+  <material name="white">
+    <color rgba="1.0 1.0 1.0 1.0"/>
+  </material>
   <!-- Transmission macro -->
   <xacro:macro name="SimpleTransmission" params="joint n">
@@ -34,17 +63,17 @@
   <!-- link 1 -->
   <link name="link1">
-    <collision>
-      <origin xyz="0 0 0" rpy="0 0 0"/>
-      <geometry>
-        <mesh filename="package://open_manipulator_pro_description/meshes/link_1.stl" scale="0.001 0.001 0.001"/>
-      </geometry>
-    </collision>
-    <visual>
-      <origin xyz="0 0 0" rpy="0 0 0"/>
-      <geometry>
-        <mesh filename="package://open_manipulator_pro_description/meshes/link_1.stl" scale="0.001 0.001 0.001"/>
-      </geometry>
-      <material name="grey"/>
-    </visual>
+    <visual>
+      <origin xyz="0 0 0" rpy="0 0 0"/>
+      <geometry>
+        <mesh filename="package://open_manipulator_pro_description/meshes/link1.stl" scale="0.001 0.001 0.001"/>
+      </geometry>
+      <material name="grey"/>
+    </visual>
+    <collision>
+      <origin xyz="0 0 0" rpy="0 0 0"/>
+      <geometry>
+        <mesh filename="package://open_manipulator_pro_description/meshes/link1.stl" scale="0.001 0.001 0.001"/>
+      </geometry>
+    </collision>
     <inertial>
       <origin xyz="0.00023 0.00000 0.06223" rpy="0 0 0"/>
@@ -60,5 +89,5 @@
     <origin xyz="0.0 0.0 0.126" rpy="0 0 0"/>
     <axis xyz="0 0 1"/>
-    <limit velocity="6.5" effort="1000" lower="${-pi*0.5}" upper="${pi*0.5}" />
+    <limit velocity="6.5" effort="1000" lower="-1.57079632679" upper="1.57079632679" />
     <dynamics damping="0.7"/>
   </joint>
@@ -67,17 +96,17 @@
   <!-- link 2 -->
   <link name="link2">
-    <collision>
-      <origin xyz="0 0 0" rpy="0 0 0"/>
-      <geometry>
-        <mesh filename="package://open_manipulator_pro_description/meshes/link_2.stl" scale="0.001 0.001 0.001"/>
-      </geometry>
-    </collision>
-    <visual>
-      <origin xyz="0 0 0" rpy="0 0 0"/>
-      <geometry>
-        <mesh filename="package://open_manipulator_pro_description/meshes/link_2.stl" scale="0.001 0.001 0.001"/>
-      </geometry>
-      <material name="grey"/>
-    </visual>
+    <visual>
+      <origin xyz="0 0 0" rpy="0 0 0"/>
+      <geometry>
+        <mesh filename="package://open_manipulator_pro_description/meshes/link2.stl" scale="0.001 0.001 0.001"/>
+      </geometry>
+      <material name="grey"/>
+    </visual>
+    <collision>
+      <origin xyz="0 0 0" rpy="0 0 0"/>
+      <geometry>
+        <mesh filename="package://open_manipulator_pro_description/meshes/link2.stl" scale="0.001 0.001 0.001"/>
+      </geometry>
+    </collision>
     <inertial>
       <origin xyz="0.00000 0.00080 0.03183" rpy="0 0 0"/>
@@ -94,5 +123,5 @@
     <origin xyz="0.0 0.0 0.033" rpy="0 0 0"/>
     <axis xyz="0 1 0"/>
-    <limit velocity="6.5" effort="1000" lower="${-pi*0.5}" upper="${pi*0.5}" />
+    <limit velocity="6.5" effort="1000" lower="-1.57079632679" upper="1.57079632679" />
     <dynamics damping="0.7"/>
   </joint>
@@ -101,17 +130,17 @@
   <!-- link 3 -->
   <link name="link3">
-    <collision>
+    <visual>
       <origin xyz="0 0.069 0" rpy="0 0 0"/>
       <geometry>
-        <mesh filename="package://open_manipulator_pro_description/meshes/link_3.stl" scale="0.001 0.001 0.001"/>
-      </geometry>
-    </collision>
-    <visual>
+        <mesh filename="package://open_manipulator_pro_description/meshes/link3.stl" scale="0.001 0.001 0.001"/>
+      </geometry>
+      <material name="grey"/>
+    </visual>
+    <collision>
       <origin xyz="0 0.069 0" rpy="0 0 0"/>
       <geometry>
-        <mesh filename="package://open_manipulator_pro_description/meshes/link_3.stl" scale="0.001 0.001 0.001"/>
-      </geometry>
-      <material name="grey"/>
-    </visual>
+        <mesh filename="package://open_manipulator_pro_description/meshes/link3.stl" scale="0.001 0.001 0.001"/>
+      </geometry>
+    </collision>
     <inertial>
       <origin xyz="0.01768 0.00019 0.20524" rpy="0 0 0"/>
@@ -127,5 +156,5 @@
     <origin xyz="0.03000 0.0 0.26400" rpy="0 0 0"/>
     <axis xyz="0 1 0"/>
-    <limit velocity="6.5" effort="1000" lower="${-pi*0.5}" upper="${pi*0.5}" />
+    <limit velocity="6.5" effort="1000" lower="-1.57079632679" upper="1.57079632679" />
     <dynamics damping="0.7"/>
   </joint>
@@ -134,17 +163,17 @@
   <!-- link 4 -->
   <link name="link4">
-    <collision>
+    <visual>
       <origin xyz="0 0.05750 0" rpy="0 0 0"/>
       <geometry>
-        <mesh filename="package://open_manipulator_pro_description/meshes/link_4.stl" scale="0.001 0.001 0.001"/>
-      </geometry>
-    </collision>
-    <visual>
+        <mesh filename="package://open_manipulator_pro_description/meshes/link4.stl" scale="0.001 0.001 0.001"/>
+      </geometry>
+      <material name="grey"/>
+    </visual>
+    <collision>
       <origin xyz="0 0.05750 0" rpy="0 0 0"/>
       <geometry>
-        <mesh filename="package://open_manipulator_pro_description/meshes/link_4.stl" scale="0.001 0.001 0.001"/>
-      </geometry>
-      <material name="grey"/>
-    </visual>
+        <mesh filename="package://open_manipulator_pro_description/meshes/link4.stl" scale="0.001 0.001 0.001"/>
+      </geometry>
+    </collision>
     <inertial>
       <origin xyz="-0.07025 0.00034 -0.00021" rpy="0 0 0"/>
@@ -160,5 +189,5 @@
     <origin xyz="0.19500 0.0 0.03000" rpy="0 0 0"/>
     <axis xyz="1 0 0"/>
-    <limit velocity="6.5" effort="1000" lower="${-pi*0.5}" upper="${pi*0.5}" />
+    <limit velocity="6.5" effort="1000" lower="-1.57079632679" upper="1.57079632679" />
     <dynamics damping="0.7"/>
   </joint>
@@ -167,17 +196,17 @@
   <!-- link 5 -->
   <link name="link5">
-    <collision>
-      <origin xyz="0 0 0" rpy="0 0 0"/>
-      <geometry>
-        <mesh filename="package://open_manipulator_pro_description/meshes/link_5.stl" scale="0.001 0.001 0.001"/>
-      </geometry>
-    </collision>
-    <visual>
-      <origin xyz="0 0 0" rpy="0 0 0"/>
-      <geometry>
-        <mesh filename="package://open_manipulator_pro_description/meshes/link_5.stl" scale="0.001 0.001 0.001"/>
-      </geometry>
-      <material name="grey"/>
-    </visual>
+    <visual>
+      <origin xyz="0 0 0" rpy="0 0 0"/>
+      <geometry>
+        <mesh filename="package://open_manipulator_pro_description/meshes/link5.stl" scale="0.001 0.001 0.001"/>
+      </geometry>
+      <material name="grey"/>
+    </visual>
+    <collision>
+      <origin xyz="0 0 0" rpy="0 0 0"/>
+      <geometry>
+        <mesh filename="package://open_manipulator_pro_description/meshes/link5.stl" scale="0.001 0.001 0.001"/>
+      </geometry>
+    </collision>
     <inertial>
       <origin xyz="0.05642 -0.00217 0.00002" rpy="0 0 0"/>
@@ -194,5 +223,5 @@
     <origin xyz="0.06300 0.00 0.00000" rpy="0 0 0"/>
     <axis xyz="0 1 0"/>
-    <limit velocity="6.5" effort="1000" lower="${-pi*0.5}" upper="${pi*0.5}" />
+    <limit velocity="6.5" effort="1000" lower="-1.57079632679" upper="1.57079632679" />
     <dynamics damping="0.7"/>
   </joint>
@@ -201,17 +230,17 @@
   <!-- link 6 -->
   <link name="link6">
-    <collision>
+    <visual>
       <origin xyz="0 0.04500 0" rpy="0 0 0"/>
       <geometry>
-        <mesh filename="package://open_manipulator_pro_description/meshes/link_6.stl" scale="0.001 0.001 0.001"/>
-      </geometry>
-    </collision>
-    <visual>
+        <mesh filename="package://open_manipulator_pro_description/meshes/link6.stl" scale="0.001 0.001 0.001"/>
+      </geometry>
+      <material name="grey"/>
+    </visual>
+    <collision>
       <origin xyz="0 0.04500 0" rpy="0 0 0"/>
       <geometry>
-        <mesh filename="package://open_manipulator_pro_description/meshes/link_6.stl" scale="0.001 0.001 0.001"/>
-      </geometry>
-      <material name="grey"/>
-    </visual>
+        <mesh filename="package://open_manipulator_pro_description/meshes/link6.stl" scale="0.001 0.001 0.001"/>
+      </geometry>
+    </collision>
     <inertial>
       <!-- <origin xyz="0.06831 -0.04457 0.00000" rpy="0 0 0"/> -->
@@ -228,5 +257,5 @@
     <origin xyz="0.12300 0.000 0.00000" rpy="0 0 0"/>
     <axis xyz="1 0 0"/>
-    <limit velocity="6.5" effort="1000" lower="${-pi*0.5}" upper="${pi*0.5}" />
+    <limit velocity="6.5" effort="1000" lower="-1.57079632679" upper="1.57079632679" />
     <dynamics damping="0.7"/>
   </joint>
@@ -235,17 +264,17 @@
   <!-- end link -->
   <link name="end_link">
-    <collision>
+    <visual>
       <origin xyz="0 0 0" rpy="0 0 0"/>
       <geometry>
         <mesh filename="package://open_manipulator_pro_description/meshes/end_link.stl" scale="0.001 0.001 0.001"/>
       </geometry>
-    </collision>
-    <visual>
+      <material name="grey"/>
+    </visual>
+    <collision>
       <origin xyz="0 0 0" rpy="0 0 0"/>
       <geometry>
         <mesh filename="package://open_manipulator_pro_description/meshes/end_link.stl" scale="0.001 0.001 0.001"/>
       </geometry>
-      <material name="grey"/>
-    </visual>
+    </collision>
     <inertial>
       <origin xyz="0.00337 0.00000 0.00000" rpy="0 0 0"/>
