Commit message: modified urdf files

File: open_manipulator_p_description/urdf/open_manipulator_p_with_gripper.gazebo.xacro (robot description, xacro)
@@ -33,8 +33,8 @@
   <!-- gripper_link -->
   <RefLink ref="gripper_link"/>
-  <!-- gripper_link_sub -->
+  <!-- gripper_sub_link -->
   <RefLink ref="gripper_sub_link"/>
-  <!-- end effector link -->
-  <gazebo reference="end_effector">
+  <!-- end_effector_link -->
+  <gazebo reference="end_effector_link">
     <material>Gazebo/Red</material>
   </gazebo>

File: open_manipulator_p_description/urdf/open_manipulator_p_with_gripper.urdf.xacro (robot description, xacro)
@@ -282,4 +282,5 @@
     <limit velocity="6.5" effort="1000" lower="0.0" upper="${740.0/2048.0*pi}" />
     <dynamics damping="0.1" friction="0.0" />
+    <mimic joint="gripper" multiplier="1"/>
   </joint>
   <!-- gripper 1 link -->
@@ -306,11 +307,11 @@
   </link>
   <!-- gripper main fixed joint-->
-  <joint name="gripper_main_fixed" type="fixed">
+  <joint name="end_effector_joint" type="fixed">
     <parent link="gripper_main_link"/>
-    <child link="end_effector"/>
+    <child link="end_effector_link"/>
     <origin xyz="0.14 0.0 0.0" rpy="0 0 0" />
   </joint>
   <!-- End Effector -->
-  <link name="end_effector">
+  <link name="end_effector_link">
     <visual>
       <origin xyz="0.0 0.0 0.0" rpy="0 0 0" />

Commit message: added camera to urdf file

File: open_manipulator_p_description/urdf/open_manipulator_p_with_gripper.gazebo.xacro (robot description, xacro)
@@ -54,3 +54,43 @@
     </plugin>
   </gazebo>
+  <!-- camera -->
+  <gazebo reference="camera_link">
+    <sensor type="camera" name="intel_realsense_r200">
+      <update_rate>30.0</update_rate>
+      <camera name="head">
+        <horizontal_fov>1.02974</horizontal_fov>
+        <image>
+          <width>1920</width>
+          <height>1080</height>
+          <format>R8G8B8</format>
+        </image>
+        <clip>
+          <near>0.02</near>
+          <far>300</far>
+        </clip>
+        <noise>
+          <type>gaussian</type>
+          <!-- Noise is sampled independently per pixel on each frame.
+               That pixel's noise value is added to each of its color
+               channels, which at that point lie in the range [0,1]. -->
+          <mean>0.0</mean>
+          <stddev>0.007</stddev>
+        </noise>
+      </camera>
+      <plugin name="camera_controller" filename="libgazebo_ros_camera.so">
+        <alwaysOn>true</alwaysOn>
+        <updateRate>0.0</updateRate>
+        <cameraName>camera/color</cameraName>
+        <imageTopicName>image_raw</imageTopicName>
+        <cameraInfoTopicName>camera_info</cameraInfoTopicName>
+        <frameName>camera_link</frameName>
+        <hackBaseline>0.07</hackBaseline>
+        <distortionK1>0.0</distortionK1>
+        <distortionK2>0.0</distortionK2>
+        <distortionK3>0.0</distortionK3>
+        <distortionT1>0.0</distortionT1>
+        <distortionT2>0.0</distortionT2>
+      </plugin>
+    </sensor>
+  </gazebo>
 </robot>

File: open_manipulator_p_description/urdf/open_manipulator_p_with_gripper.urdf.xacro (robot description, xacro)
@@ -325,3 +325,11 @@
     </inertial>
   </link>
+  <!-- Realsense Camera Joint Position -->
+  <joint name="camera_joint" type="fixed">
+    <axis xyz="0 1 0" />
+    <origin xyz="0.070 0.032 0.052" rpy="0 0 0"/>
+    <parent link="gripper_main_link"/>
+    <child link="camera_link"/>
+  </joint>
+  <link name="camera_link"/>
 </robot>
