Commit message: updated urdf related files

File: open_manipulator_p_description/urdf/open_manipulator_p.gazebo.xacro (robot description, xacro)
@@ -1,55 +1,46 @@
 <?xml version="1.0"?>
-<robot>
+<robot xmlns:xacro="http://ros.org/wiki/xacro">
+  <!-- Gazebo Reference macro -->
+  <xacro:macro name="RefLink" params="ref">
+    <gazebo reference="${ref}">
+      <kp>1000000.0</kp>
+      <kd>100.0</kd>
+      <mu1>30.0</mu1>
+      <mu2>30.0</mu2>
+      <maxVel>1.0</maxVel>
+      <minDepth>0.001</minDepth>
+      <material>Gazebo/DarkGrey</material>
+    </gazebo>
+  </xacro:macro>
+  <!-- World -->
+  <gazebo reference="world"/>
+  <!-- Link1 -->
+  <RefLink ref="link1"/>
+  <!-- Link2 -->
+  <RefLink ref="link2"/>
+  <!-- Link3 -->
+  <RefLink ref="link3"/>
+  <!-- Link4 -->
+  <RefLink ref="link4"/>
+  <!-- Link5 -->
+  <RefLink ref="link5"/>
+  <!-- Link6 -->
+  <RefLink ref="link6"/>
+  <!-- end_link -->
+  <RefLink ref="end_link"/>
   <!-- ros_control plugin -->
   <gazebo>
     <plugin name="gazebo_ros_control" filename="libgazebo_ros_control.so">
-      <robotNamespace>open_manipulator_p</robotNamespace>
       <robotSimType>gazebo_ros_control/DefaultRobotHWSim</robotSimType>
     </plugin>
   </gazebo>
-  <!-- World -->
-  <gazebo reference="world">
-  </gazebo>
-  <!-- Link1 -->
-  <gazebo reference="link1">
-    <mu1>0.2</mu1>
-    <mu2>0.2</mu2>
-    <material>Gazebo/Grey</material>
-  </gazebo>
-  <!-- Link2 -->
-  <gazebo reference="link2">
-    <mu1>0.2</mu1>
-    <mu2>0.2</mu2>
-    <material>Gazebo/Grey</material>
-  </gazebo>
-  <!-- Link3 -->
-  <gazebo reference="link3">
-    <mu1>0.2</mu1>
-    <mu2>0.2</mu2>
-    <material>Gazebo/Grey</material>
-  </gazebo>
-  <!-- Link4 -->
-  <gazebo reference="link4">
-    <mu1>0.2</mu1>
-    <mu2>0.2</mu2>
-    <material>Gazebo/Grey</material>
-  </gazebo>
-  <!-- Link5 -->
-  <gazebo reference="link5">
-    <mu1>0.2</mu1>
-    <mu2>0.2</mu2>
-    <material>Gazebo/Grey</material>
-  </gazebo>
-  <!-- Link6 -->
-  <gazebo reference="link6">
-    <mu1>0.2</mu1>
-    <mu2>0.2</mu2>
-    <material>Gazebo/Grey</material>
-  </gazebo>
-  <!-- End Link -->
-  <gazebo reference="end_link">
-    <mu1>0.2</mu1>
-    <mu2>0.2</mu2>
-    <material>Gazebo/Grey</material>
+  <gazebo>
+    <!-- loading plugin: mimic joints works in gazebo now -->
+    <plugin name="gazebo_gripper_ros_control" filename="libroboticsgroup_gazebo_mimic_joint_plugin.so">
+      <joint>gripper</joint>
+      <mimicJoint>gripper_sub</mimicJoint>
+      <multiplier>1.0</multiplier>
+      <offset>0.0</offset>
+    </plugin>
   </gazebo>
 </robot>

File: open_manipulator_p_description/urdf/open_manipulator_p.urdf.xacro (robot description, xacro)
@@ -1,33 +1,4 @@
 <?xml version="1.0"?>
-<!-- Revolute-Revolute Manipulator -->
-<robot name="open_manipulator_p" xmlns:xacro="http://www.ros.org/wiki/xacro">
-  <!-- some parameters -->
-  <xacro:property name="pi" value="3.141592654" />
-  <!-- Import all Gazebo-customization elements, including Gazebo colors -->
-  <xacro:include filename="$(find open_manipulator_p_description)/urdf/open_manipulator_p.gazebo.xacro" />
-  <!-- Import Rviz colors -->
-  <xacro:include filename="$(find open_manipulator_p_description)/urdf/materials.xacro" />
-  <!-- Transmission macro -->
-  <xacro:macro name="SimpleTransmission" params="joint n">
-    <transmission name="tran${n}">
-      <type>transmission_interface/SimpleTransmission</type>
-      <joint name="${joint}">
-        <hardwareInterface>hardware_interface/PositionJointInterface</hardwareInterface>
-      </joint>
-      <actuator name="motor${n}">
-        <hardwareInterface>hardware_interface/PositionJointInterface</hardwareInterface>
-        <mechanicalReduction>1</mechanicalReduction>
-      </actuator>
-    </transmission>
-  </xacro:macro>
-  <!-- World -->
-  <link name="world">
-  </link>
-  <!-- World fixed joint-->
-  <joint name="world_fixed" type="fixed">
-    <origin xyz="0 0 0" rpy="0 0 0"/>
-    <parent link="world"/>
-    <child link="link1"/>
-  </joint>
+<robot xmlns:xacro="http://www.ros.org/wiki/xacro">
   <!-- link 1 -->
   <link name="link1">
@@ -61,6 +32,4 @@
     <dynamics damping="0.7"/>
   </joint>
-  <!-- Transmission 1 -->
-  <xacro:SimpleTransmission n="1" joint="joint1" />
   <!-- link 2 -->
   <link name="link2">
@@ -90,15 +59,13 @@
     <parent link="link2"/>
     <child link="link3"/>
-    <origin xyz="0.0 0.0 0.033" rpy="0 0 0"/>
+    <origin xyz="0.0 0.069 0.033" rpy="0 0 0"/>
     <axis xyz="0 1 0"/>
     <limit velocity="6.5" effort="1000" lower="${-pi*0.5}" upper="${pi*0.5}" />
     <dynamics damping="0.7"/>
   </joint>
-  <!-- Transmission 2 -->
-  <xacro:SimpleTransmission n="2" joint="joint2" />
   <!-- link 3 -->
   <link name="link3">
     <collision>
-      <origin xyz="0 0.069 0" rpy="0 0 0"/>
+      <origin xyz="0 0 0" rpy="0 0 0"/>
       <geometry>
         <mesh filename="package://open_manipulator_p_description/meshes/link_3.stl" scale="0.001 0.001 0.001"/>
@@ -106,5 +73,5 @@
     </collision>
     <visual>
-      <origin xyz="0 0.069 0" rpy="0 0 0"/>
+      <origin xyz="0 0 0" rpy="0 0 0"/>
       <geometry>
         <mesh filename="package://open_manipulator_p_description/meshes/link_3.stl" scale="0.001 0.001 0.001"/>
@@ -113,5 +80,6 @@
     </visual>
     <inertial>
-      <origin xyz="0.01768 0.00019 0.20524" rpy="0 0 0"/>
+      <origin xyz="0.01768 -0.06881 0.20524" rpy="0 0 0"/>
+      <!--<origin xyz="-0.01232 -0.05731 -0.05876" rpy="0 0 0"/>-->
       <mass value="1.30260"/>
       <inertia ixx="1.0" ixy="0.0" ixz="0.0" iyy="1.0" iyz="0.0" izz="1.0" />
@@ -123,15 +91,13 @@
     <parent link="link3"/>
     <child link="link4"/>
-    <origin xyz="0.03000 0.0 0.26400" rpy="0 0 0"/>
+    <origin xyz="0.03000 -0.01150 0.26400" rpy="0 0 0"/>
     <axis xyz="0 1 0"/>
     <limit velocity="6.5" effort="1000" lower="${-pi*0.5}" upper="${pi*0.5}" />
     <dynamics damping="0.7"/>
   </joint>
-  <!-- Transmission 3 -->
-  <xacro:SimpleTransmission n="3" joint="joint3" />
   <!-- link 4 -->
   <link name="link4">
     <collision>
-      <origin xyz="0 0.05750 0" rpy="0 0 0"/>
+      <origin xyz="0 0 0" rpy="0 0 0"/>
       <geometry>
         <mesh filename="package://open_manipulator_p_description/meshes/link_4.stl" scale="0.001 0.001 0.001"/>
@@ -139,5 +105,5 @@
     </collision>
     <visual>
-      <origin xyz="0 0.05750 0" rpy="0 0 0"/>
+      <origin xyz="0 0 0" rpy="0 0 0"/>
       <geometry>
         <mesh filename="package://open_manipulator_p_description/meshes/link_4.stl" scale="0.001 0.001 0.001"/>
@@ -146,5 +112,6 @@
     </visual>
     <inertial>
-      <origin xyz="-0.07025 0.00034 -0.00021" rpy="0 0 0"/>
+      <origin xyz="0.12475 -0.05716 0.02979" rpy="0 0 0"/>
+      <!--<origin xyz="-0.07025 0.00034 -0.00021" rpy="0 0 0"/>-->
       <mass value="1.15977"/>
       <inertia ixx="1.0" ixy="0.0" ixz="0.0" iyy="1.0" iyz="0.0" izz="1.0" />
@@ -156,11 +123,9 @@
     <parent link="link4"/>
     <child link="link5"/>
-    <origin xyz="0.19500 0.0 0.03000" rpy="0 0 0"/>
+    <origin xyz="0.19500 -0.05750 0.03000" rpy="0 0 0"/>
     <axis xyz="1 0 0"/>
     <limit velocity="6.5" effort="1000" lower="${-pi*0.5}" upper="${pi*0.5}" />
     <dynamics damping="0.7"/>
   </joint>
-  <!-- Transmission 4 -->
-  <xacro:SimpleTransmission n="4" joint="joint4" />
   <!-- link 5 -->
   <link name="link5">
@@ -190,15 +155,13 @@
     <parent link="link5"/>
     <child link="link6"/>
-    <origin xyz="0.06300 0.00 0.00000" rpy="0 0 0"/>
+    <origin xyz="0.06300 0.04500 0.00000" rpy="0 0 0"/>
     <axis xyz="0 1 0"/>
     <limit velocity="6.5" effort="1000" lower="${-pi*0.5}" upper="${pi*0.5}" />
     <dynamics damping="0.7"/>
   </joint>
-  <!-- Transmission 5 -->
-  <xacro:SimpleTransmission n="5" joint="joint5" />
   <!-- link 6 -->
   <link name="link6">
     <collision>
-      <origin xyz="0 0.04500 0" rpy="0 0 0"/>
+      <origin xyz="0 0 0" rpy="0 0 0"/>
       <geometry>
         <mesh filename="package://open_manipulator_p_description/meshes/link_6.stl" scale="0.001 0.001 0.001"/>
@@ -206,5 +169,5 @@
     </collision>
     <visual>
-      <origin xyz="0 0.04500 0" rpy="0 0 0"/>
+      <origin xyz="0 0 0" rpy="0 0 0"/>
       <geometry>
         <mesh filename="package://open_manipulator_p_description/meshes/link_6.stl" scale="0.001 0.001 0.001"/>
@@ -213,6 +176,6 @@
     </visual>
     <inertial>
-      <!-- <origin xyz="0.06831 -0.04457 0.00000" rpy="0 0 0"/> -->
-      <origin xyz="-0.05469 0.00043 0.00000" rpy="0 0 0"/>
+      <origin xyz="0.06831 -0.04457 0.00000" rpy="0 0 0"/>
+      <!--<origin xyz="-0.05469 0.00043 0.00000" rpy="0 0 0"/>-->
       <mass value="0.43273"/>
       <inertia ixx="1.0" ixy="0.0" ixz="0.0" iyy="1.0" iyz="0.0" izz="1.0" />
@@ -224,26 +187,24 @@
     <parent link="link6"/>
     <child link="end_link"/>
-    <origin xyz="0.12300 0.000 0.00000" rpy="0 0 0"/>
+    <origin xyz="0.12300 -0.04500 0.00000" rpy="0 0 0"/>
     <axis xyz="1 0 0"/>
     <limit velocity="6.5" effort="1000" lower="${-pi*0.5}" upper="${pi*0.5}" />
     <dynamics damping="0.7"/>
   </joint>
-  <!-- Transmission 6 -->
-  <xacro:SimpleTransmission n="6" joint="joint6" />
   <!-- end link -->
   <link name="end_link">
-    <collision>
-      <origin xyz="0 0 0" rpy="0 0 0"/>
+    <visual>
+      <origin xyz="0.0 0.0 0.0" rpy="0 0 0" />
       <geometry>
         <mesh filename="package://open_manipulator_p_description/meshes/end_link.stl" scale="0.001 0.001 0.001"/>
       </geometry>
-    </collision>
-    <visual>
-      <origin xyz="0 0 0" rpy="0 0 0"/>
+      <material name="grey"/>
+    </visual>
+    <collision>
+      <origin xyz="0.0 0.0 0.0" rpy="0 0 0" />
       <geometry>
         <mesh filename="package://open_manipulator_p_description/meshes/end_link.stl" scale="0.001 0.001 0.001"/>
       </geometry>
-      <material name="grey"/>
-    </visual>
+    </collision>
     <inertial>
       <origin xyz="0.00337 0.00000 0.00000" rpy="0 0 0"/>

File: open_manipulator_p_description/urdf/open_manipulator_p_with_gripper.gazebo.xacro (robot description, xacro)
@@ -1,73 +1,56 @@
 <?xml version="1.0"?>
-<robot>
+<robot xmlns:xacro="http://ros.org/wiki/xacro">
+  <!-- Gazebo Reference macro -->
+  <xacro:macro name="RefLink" params="ref">
+    <gazebo reference="${ref}">
+      <kp>1000000.0</kp>
+      <kd>100.0</kd>
+      <mu1>30.0</mu1>
+      <mu2>30.0</mu2>
+      <maxVel>1.0</maxVel>
+      <minDepth>0.001</minDepth>
+      <material>Gazebo/DarkGrey</material>
+    </gazebo>
+  </xacro:macro>
+  <!-- World -->
+  <gazebo reference="world"/>
+  <!-- Link1 -->
+  <RefLink ref="link1"/>
+  <!-- Link2 -->
+  <RefLink ref="link2"/>
+  <!-- Link3 -->
+  <RefLink ref="link3"/>
+  <!-- Link4 -->
+  <RefLink ref="link4"/>
+  <!-- Link5 -->
+  <RefLink ref="link5"/>
+  <!-- Link6 -->
+  <RefLink ref="link6"/>
+  <!-- end_link -->
+  <RefLink ref="end_link"/>
+  <!-- gripper_main_link -->
+  <RefLink ref="gripper_main_link"/>
+  <!-- gripper_link -->
+  <RefLink ref="gripper_link"/>
+  <!-- gripper_link_sub -->
+  <RefLink ref="gripper_sub_link"/>
+  <!-- end effector link -->
+  <gazebo reference="end_effector">
+    <material>Gazebo/Red</material>
+  </gazebo>
   <!-- ros_control plugin -->
   <gazebo>
     <plugin name="gazebo_ros_control" filename="libgazebo_ros_control.so">
-      <robotNamespace>open_manipulator_p</robotNamespace>
       <robotSimType>gazebo_ros_control/DefaultRobotHWSim</robotSimType>
     </plugin>
   </gazebo>
-  <!-- World -->
-  <gazebo reference="world">
-  </gazebo>
-  <!-- Link1 -->
-  <gazebo reference="link1">
-    <mu1>0.2</mu1>
-    <mu2>0.2</mu2>
-    <material>Gazebo/Grey</material>
-  </gazebo>
-  <!-- Link2 -->
-  <gazebo reference="link2">
-    <mu1>0.2</mu1>
-    <mu2>0.2</mu2>
-    <material>Gazebo/Grey</material>
-  </gazebo>
-  <!-- Link3 -->
-  <gazebo reference="link3">
-    <mu1>0.2</mu1>
-    <mu2>0.2</mu2>
-    <material>Gazebo/Grey</material>
-  </gazebo>
-  <!-- Link4 -->
-  <gazebo reference="link4">
-    <mu1>0.2</mu1>
-    <mu2>0.2</mu2>
-    <material>Gazebo/Grey</material>
-  </gazebo>
-  <!-- Link5 -->
-  <gazebo reference="link5">
-    <mu1>0.2</mu1>
-    <mu2>0.2</mu2>
-    <material>Gazebo/Grey</material>
-  </gazebo>
-  <!-- Link6 -->
-  <gazebo reference="link6">
-    <mu1>0.2</mu1>
-    <mu2>0.2</mu2>
-    <material>Gazebo/Grey</material>
-  </gazebo>
-  <!-- gripper main link -->
-  <gazebo reference="gripper_main_link">
-    <mu1>0.2</mu1>
-    <mu2>0.2</mu2>
-    <material>Gazebo/Grey</material>
-  </gazebo>
-  <!-- gripper link -->
-  <gazebo reference="gripper_link">
-    <mu1>0.2</mu1>
-    <mu2>0.2</mu2>
-    <material>Gazebo/Grey</material>
-  </gazebo>
-  <!-- gripper 1 link -->
-  <gazebo reference="gripper_sub_link">
-    <mu1>0.2</mu1>
-    <mu2>0.2</mu2>
-    <material>Gazebo/Grey</material>
-  </gazebo>
-  <!-- End Effector -->
-  <gazebo reference="end_effector">
-    <mu1>0.2</mu1>
-    <mu2>0.2</mu2>
-    <material>Gazebo/Red</material>
+  <gazebo>
+    <!-- loading plugin: mimic joints works in gazebo now -->
+    <plugin name="gazebo_gripper_ros_control" filename="libroboticsgroup_gazebo_mimic_joint_plugin.so">
+      <joint>gripper</joint>
+      <mimicJoint>gripper_sub</mimicJoint>
+      <multiplier>1.0</multiplier>
+      <offset>0.0</offset>
+    </plugin>
   </gazebo>
 </robot>

File: open_manipulator_p_description/urdf/open_manipulator_p_with_gripper.urdf.xacro (robot description, xacro)
@@ -1,35 +1,4 @@
 <?xml version="1.0"?>
-<!-- Revolute-Revolute Manipulator -->
-<robot name="open_manipulator_p" xmlns:xacro="http://www.ros.org/wiki/xacro">
-  <!-- some parameters -->
-  <xacro:property name="pi" value="3.141592654" />
-  <!-- some parameters -->
-  <xacro:property name="pi" value="3.141592654" />
-  <!-- Import all Gazebo-customization elements, including Gazebo colors -->
-  <xacro:include filename="$(find open_manipulator_p_description)/urdf/open_manipulator_p_with_gripper.gazebo.xacro" />
-  <!-- Import Rviz colors -->
-  <xacro:include filename="$(find open_manipulator_p_description)/urdf/materials.xacro" />
-  <!-- Transmission macro -->
-  <xacro:macro name="SimpleTransmission" params="joint n">
-    <transmission name="tran${n}">
-      <type>transmission_interface/SimpleTransmission</type>
-      <joint name="${joint}">
-        <hardwareInterface>hardware_interface/PositionJointInterface</hardwareInterface>
-      </joint>
-      <actuator name="motor${n}">
-        <hardwareInterface>hardware_interface/PositionJointInterface</hardwareInterface>
-        <mechanicalReduction>1</mechanicalReduction>
-      </actuator>
-    </transmission>
-  </xacro:macro>
-  <!-- World -->
-  <link name="world">
-  </link>
-  <!-- World fixed joint-->
-  <joint name="world_fixed" type="fixed">
-    <origin xyz="0 0 0" rpy="0 0 0"/>
-    <parent link="world"/>
-    <child link="link1"/>
-  </joint>
+<robot xmlns:xacro="http://www.ros.org/wiki/xacro">
   <!-- link 1 -->
   <link name="link1">
@@ -63,6 +32,4 @@
     <dynamics damping="0.7"/>
   </joint>
-  <!-- Transmission 1 -->
-  <xacro:SimpleTransmission n="1" joint="joint1" />
   <!-- link 2 -->
   <link name="link2">
@@ -97,6 +64,4 @@
     <dynamics damping="0.7"/>
   </joint>
-  <!-- Transmission 2 -->
-  <xacro:SimpleTransmission n="2" joint="joint2" />
   <!-- link 3 -->
   <link name="link3">
@@ -131,6 +96,4 @@
     <dynamics damping="0.7"/>
   </joint>
-  <!-- Transmission 3 -->
-  <xacro:SimpleTransmission n="3" joint="joint3" />
   <!-- link 4 -->
   <link name="link4">
@@ -165,6 +128,4 @@
     <dynamics damping="0.7"/>
   </joint>
-  <!-- Transmission 4 -->
-  <xacro:SimpleTransmission n="4" joint="joint4" />
   <!-- link 5 -->
   <link name="link5">
@@ -199,6 +160,4 @@
     <dynamics damping="0.7"/>
   </joint>
-  <!-- Transmission 5 -->
-  <xacro:SimpleTransmission n="5" joint="joint5" />
   <!-- link 6 -->
   <link name="link6">
@@ -227,5 +186,5 @@
   <joint name="joint6" type="revolute">
     <parent link="link6"/>
-    <child link="gripper_main_link"/>
+    <child link="end_link"/>
     <origin xyz="0.12300 -0.04500 0.00000" rpy="0 0 0"/>
     <axis xyz="1 0 0"/>
@@ -233,6 +192,32 @@
     <dynamics damping="0.7"/>
   </joint>
-  <!-- Transmission 6 -->
-  <xacro:SimpleTransmission n="6" joint="joint6" />
+  <!-- end link -->
+  <link name="end_link">
+    <visual>
+      <origin xyz="0.0 0.0 0.0" rpy="0 0 0" />
+      <geometry>
+        <mesh filename="package://open_manipulator_p_description/meshes/end_link.stl" scale="0.001 0.001 0.001"/>
+      </geometry>
+      <material name="grey"/>
+    </visual>
+    <collision>
+      <origin xyz="0.0 0.0 0.0" rpy="0 0 0" />
+      <geometry>
+        <mesh filename="package://open_manipulator_p_description/meshes/end_link.stl" scale="0.001 0.001 0.001"/>
+      </geometry>
+    </collision>
+    <inertial>
+      <origin xyz="0.00337 0.00000 0.00000" rpy="0 0 0"/>
+      <mass value="0.01919"/>
+      <inertia ixx="1.0" ixy="0.0" ixz="0.0" iyy="1.0" iyz="0.0" izz="1.0" />
+      <!--<inertia ixx="0.00000938" ixy="0.0" ixz="0.0" iyy="0.00000338" iyz="0.0" izz="0.00000635" />-->
+    </inertial>
+  </link>
+  <!-- gripper main fixed joint-->
+  <joint name="end_link_fixed" type="fixed">
+    <parent link="end_link"/>
+    <child link="gripper_main_link"/>
+    <origin xyz="0.007 0.0 0.0" rpy="0 0 0" />
+  </joint>
   <!-- gripper main link -->
   <link name="gripper_main_link">
@@ -266,6 +251,4 @@
     <dynamics damping="0.1" friction="0.0" />
   </joint>
-  <!-- Transmission gripper -->
-  <xacro:SimpleTransmission n="_gripper" joint="gripper" />
   <!-- gripper link -->
   <link name="gripper_link">
@@ -300,6 +283,4 @@
     <dynamics damping="0.1" friction="0.0" />
   </joint>
-  <!-- Transmission gripper -->
-  <xacro:SimpleTransmission n="_gripper_sub" joint="gripper_sub" />
   <!-- gripper 1 link -->
   <link name="gripper_sub_link">

Commit message: switched gripper open and close

File: open_manipulator_p_description/urdf/open_manipulator_p.gazebo.xacro (robot description, xacro)
@@ -35,12 +35,3 @@
     </plugin>
   </gazebo>
-  <gazebo>
-    <!-- loading plugin: mimic joints works in gazebo now -->
-    <plugin name="gazebo_gripper_ros_control" filename="libroboticsgroup_gazebo_mimic_joint_plugin.so">
-      <joint>gripper</joint>
-      <mimicJoint>gripper_sub</mimicJoint>
-      <multiplier>1.0</multiplier>
-      <offset>0.0</offset>
-    </plugin>
-  </gazebo>
 </robot>

File: open_manipulator_p_description/urdf/open_manipulator_p_with_gripper.urdf.xacro (robot description, xacro)
@@ -243,10 +243,9 @@
   <!-- gripper joint -->
   <joint name="gripper" type="revolute">
-    <axis xyz="0 0 -1" />
-    <origin xyz="0.0552 -0.0460 0" rpy="0 0 ${45.0*pi/180.0}"/>
-    <!-- <origin xyz="0.0552 -0.0370 0" rpy="0 0 0"/> -->
+    <axis xyz="0 0 1" />
+    <origin xyz="0.0552 -0.0400 0" rpy="0 0 -0.4"/>
     <parent link="gripper_main_link"/>
     <child link="gripper_link"/>
-    <limit velocity="6.5" effort="1000" lower="0.0" upper="${740.0/2048.0*pi}" />
+    <limit velocity="6.5" effort="1000" lower="0.0" upper="1.1" />
     <dynamics damping="0.1" friction="0.0" />
   </joint>
@@ -275,10 +274,9 @@
   <!-- gripper joint 1 -->
   <joint name="gripper_sub" type="revolute">
-    <axis xyz="0 0 1" />
-    <origin xyz="0.0552 0.0460 0" rpy="0 0 ${-45.0*pi/180.0}"/>
-    <!-- <origin xyz="0.0552 0.0370 0" rpy="0 0 0"/> -->
+    <axis xyz="0 0 -1" />
+    <origin xyz="0.0552 0.0400 0" rpy="0 0 0.4"/>
     <parent link="gripper_main_link"/>
     <child link="gripper_sub_link"/>
-    <limit velocity="6.5" effort="1000" lower="0.0" upper="${740.0/2048.0*pi}" />
+    <limit velocity="6.5" effort="1000" lower="0.0" upper="1.1" />
     <dynamics damping="0.1" friction="0.0" />
     <mimic joint="gripper" multiplier="1"/>
