Commit message: removed unused colours

File: open_manipulator_p_description/urdf/open_manipulator_p_robot.urdf.xacro (robot description, xacro)
@@ -38,10 +38,4 @@
     <color rgba="0.5 0.5 0.5 1.0"/>
   </material>
-  <material name="orange">
-    <color rgba="${255/255} ${108/255} ${10/255} 1.0"/>
-  </material>
-  <material name="brown">
-    <color rgba="${222/255} ${207/255} ${195/255} 1.0"/>
-  </material>
   <!-- link 1 -->
   <link name="link1">

File: open_manipulator_p_description/urdf/open_manipulator_p_with_gripper_robot.urdf.xacro (robot description, xacro)
@@ -38,10 +38,4 @@
     <color rgba="0.5 0.5 0.5 1.0"/>
   </material>
-  <material name="orange">
-    <color rgba="${255/255} ${108/255} ${10/255} 1.0"/>
-  </material>
-  <material name="brown">
-    <color rgba="${222/255} ${207/255} ${195/255} 1.0"/>
-  </material>
   <!-- link 1 -->
   <link name="link1">
