Commit message: updated urdf files

File: open_manipulator_p_description/urdf/open_manipulator_p.urdf.xacro (robot description, xacro)
@@ -3,17 +3,17 @@
   <!-- link 1 -->
   <link name="link1">
-    <collision>
-      <origin xyz="0 0 0" rpy="0 0 0"/>
-      <geometry>
-        <mesh filename="package://open_manipulator_p_description/meshes/link_1.stl" scale="0.001 0.001 0.001"/>
-      </geometry>
-    </collision>
-    <visual>
-      <origin xyz="0 0 0" rpy="0 0 0"/>
-      <geometry>
-        <mesh filename="package://open_manipulator_p_description/meshes/link_1.stl" scale="0.001 0.001 0.001"/>
-      </geometry>
-      <material name="grey"/>
-    </visual>
+    <visual>
+      <origin xyz="0 0 0" rpy="0 0 0"/>
+      <geometry>
+        <mesh filename="package://open_manipulator_p_description/meshes/link1.stl" scale="0.001 0.001 0.001"/>
+      </geometry>
+      <material name="grey"/>
+    </visual>
+    <collision>
+      <origin xyz="0 0 0" rpy="0 0 0"/>
+      <geometry>
+        <mesh filename="package://open_manipulator_p_description/meshes/link1.stl" scale="0.001 0.001 0.001"/>
+      </geometry>
+    </collision>
     <inertial>
       <origin xyz="0.00023 0.00000 0.06223" rpy="0 0 0"/>
@@ -34,17 +34,17 @@
   <!-- link 2 -->
   <link name="link2">
-    <collision>
-      <origin xyz="0 0 0" rpy="0 0 0"/>
-      <geometry>
-        <mesh filename="package://open_manipulator_p_description/meshes/link_2.stl" scale="0.001 0.001 0.001"/>
-      </geometry>
-    </collision>
-    <visual>
-      <origin xyz="0 0 0" rpy="0 0 0"/>
-      <geometry>
-        <mesh filename="package://open_manipulator_p_description/meshes/link_2.stl" scale="0.001 0.001 0.001"/>
-      </geometry>
-      <material name="grey"/>
-    </visual>
+    <visual>
+      <origin xyz="0 0 0" rpy="0 0 0"/>
+      <geometry>
+        <mesh filename="package://open_manipulator_p_description/meshes/link2.stl" scale="0.001 0.001 0.001"/>
+      </geometry>
+      <material name="grey"/>
+    </visual>
+    <collision>
+      <origin xyz="0 0 0" rpy="0 0 0"/>
+      <geometry>
+        <mesh filename="package://open_manipulator_p_description/meshes/link2.stl" scale="0.001 0.001 0.001"/>
+      </geometry>
+    </collision>
     <inertial>
       <origin xyz="0.00000 0.00080 0.03183" rpy="0 0 0"/>
@@ -66,17 +66,17 @@
   <!-- link 3 -->
   <link name="link3">
-    <collision>
-      <origin xyz="0 0 0" rpy="0 0 0"/>
-      <geometry>
-        <mesh filename="package://open_manipulator_p_description/meshes/link_3.stl" scale="0.001 0.001 0.001"/>
-      </geometry>
-    </collision>
-    <visual>
-      <origin xyz="0 0 0" rpy="0 0 0"/>
-      <geometry>
-        <mesh filename="package://open_manipulator_p_description/meshes/link_3.stl" scale="0.001 0.001 0.001"/>
-      </geometry>
-      <material name="grey"/>
-    </visual>
+    <visual>
+      <origin xyz="0 0 0" rpy="0 0 0"/>
+      <geometry>
+        <mesh filename="package://open_manipulator_p_description/meshes/link3.stl" scale="0.001 0.001 0.001"/>
+      </geometry>
+      <material name="grey"/>
+    </visual>
+    <collision>
+      <origin xyz="0 0 0" rpy="0 0 0"/>
+      <geometry>
+        <mesh filename="package://open_manipulator_p_description/meshes/link3.stl" scale="0.001 0.001 0.001"/>
+      </geometry>
+    </collision>
     <inertial>
       <origin xyz="0.01768 -0.06881 0.20524" rpy="0 0 0"/>
@@ -98,17 +98,17 @@
   <!-- link 4 -->
   <link name="link4">
-    <collision>
-      <origin xyz="0 0 0" rpy="0 0 0"/>
-      <geometry>
-        <mesh filename="package://open_manipulator_p_description/meshes/link_4.stl" scale="0.001 0.001 0.001"/>
-      </geometry>
-    </collision>
-    <visual>
-      <origin xyz="0 0 0" rpy="0 0 0"/>
-      <geometry>
-        <mesh filename="package://open_manipulator_p_description/meshes/link_4.stl" scale="0.001 0.001 0.001"/>
-      </geometry>
-      <material name="grey"/>
-    </visual>
+    <visual>
+      <origin xyz="0 0 0" rpy="0 0 0"/>
+      <geometry>
+        <mesh filename="package://open_manipulator_p_description/meshes/link4.stl" scale="0.001 0.001 0.001"/>
+      </geometry>
+      <material name="grey"/>
+    </visual>
+    <collision>
+      <origin xyz="0 0 0" rpy="0 0 0"/>
+      <geometry>
+        <mesh filename="package://open_manipulator_p_description/meshes/link4.stl" scale="0.001 0.001 0.001"/>
+      </geometry>
+    </collision>
     <inertial>
       <origin xyz="0.12475 -0.05716 0.02979" rpy="0 0 0"/>
@@ -130,17 +130,17 @@
   <!-- link 5 -->
   <link name="link5">
-    <collision>
-      <origin xyz="0 0 0" rpy="0 0 0"/>
-      <geometry>
-        <mesh filename="package://open_manipulator_p_description/meshes/link_5.stl" scale="0.001 0.001 0.001"/>
-      </geometry>
-    </collision>
-    <visual>
-      <origin xyz="0 0 0" rpy="0 0 0"/>
-      <geometry>
-        <mesh filename="package://open_manipulator_p_description/meshes/link_5.stl" scale="0.001 0.001 0.001"/>
-      </geometry>
-      <material name="grey"/>
-    </visual>
+    <visual>
+      <origin xyz="0 0 0" rpy="0 0 0"/>
+      <geometry>
+        <mesh filename="package://open_manipulator_p_description/meshes/link5.stl" scale="0.001 0.001 0.001"/>
+      </geometry>
+      <material name="grey"/>
+    </visual>
+    <collision>
+      <origin xyz="0 0 0" rpy="0 0 0"/>
+      <geometry>
+        <mesh filename="package://open_manipulator_p_description/meshes/link5.stl" scale="0.001 0.001 0.001"/>
+      </geometry>
+    </collision>
     <inertial>
       <origin xyz="0.05642 -0.00217 0.00002" rpy="0 0 0"/>
@@ -162,17 +162,17 @@
   <!-- link 6 -->
   <link name="link6">
-    <collision>
-      <origin xyz="0 0 0" rpy="0 0 0"/>
-      <geometry>
-        <mesh filename="package://open_manipulator_p_description/meshes/link_6.stl" scale="0.001 0.001 0.001"/>
-      </geometry>
-    </collision>
-    <visual>
-      <origin xyz="0 0 0" rpy="0 0 0"/>
-      <geometry>
-        <mesh filename="package://open_manipulator_p_description/meshes/link_6.stl" scale="0.001 0.001 0.001"/>
-      </geometry>
-      <material name="grey"/>
-    </visual>
+    <visual>
+      <origin xyz="0 0 0" rpy="0 0 0"/>
+      <geometry>
+        <mesh filename="package://open_manipulator_p_description/meshes/link6.stl" scale="0.001 0.001 0.001"/>
+      </geometry>
+      <material name="grey"/>
+    </visual>
+    <collision>
+      <origin xyz="0 0 0" rpy="0 0 0"/>
+      <geometry>
+        <mesh filename="package://open_manipulator_p_description/meshes/link6.stl" scale="0.001 0.001 0.001"/>
+      </geometry>
+    </collision>
     <inertial>
       <origin xyz="0.06831 -0.04457 0.00000" rpy="0 0 0"/>

File: open_manipulator_p_description/urdf/open_manipulator_p_with_gripper.urdf.xacro (robot description, xacro)
@@ -3,17 +3,17 @@
   <!-- link 1 -->
   <link name="link1">
-    <collision>
-      <origin xyz="0 0 0" rpy="0 0 0"/>
-      <geometry>
-        <mesh filename="package://open_manipulator_p_description/meshes/link_1.stl" scale="0.001 0.001 0.001"/>
-      </geometry>
-    </collision>
-    <visual>
-      <origin xyz="0 0 0" rpy="0 0 0"/>
-      <geometry>
-        <mesh filename="package://open_manipulator_p_description/meshes/link_1.stl" scale="0.001 0.001 0.001"/>
-      </geometry>
-      <material name="grey"/>
-    </visual>
+    <visual>
+      <origin xyz="0 0 0" rpy="0 0 0"/>
+      <geometry>
+        <mesh filename="package://open_manipulator_p_description/meshes/link1.stl" scale="0.001 0.001 0.001"/>
+      </geometry>
+      <material name="grey"/>
+    </visual>
+    <collision>
+      <origin xyz="0 0 0" rpy="0 0 0"/>
+      <geometry>
+        <mesh filename="package://open_manipulator_p_description/meshes/link1.stl" scale="0.001 0.001 0.001"/>
+      </geometry>
+    </collision>
     <inertial>
       <origin xyz="0.00023 0.00000 0.06223" rpy="0 0 0"/>
@@ -34,17 +34,17 @@
   <!-- link 2 -->
   <link name="link2">
-    <collision>
-      <origin xyz="0 0 0" rpy="0 0 0"/>
-      <geometry>
-        <mesh filename="package://open_manipulator_p_description/meshes/link_2.stl" scale="0.001 0.001 0.001"/>
-      </geometry>
-    </collision>
-    <visual>
-      <origin xyz="0 0 0" rpy="0 0 0"/>
-      <geometry>
-        <mesh filename="package://open_manipulator_p_description/meshes/link_2.stl" scale="0.001 0.001 0.001"/>
-      </geometry>
-      <material name="grey"/>
-    </visual>
+    <visual>
+      <origin xyz="0 0 0" rpy="0 0 0"/>
+      <geometry>
+        <mesh filename="package://open_manipulator_p_description/meshes/link2.stl" scale="0.001 0.001 0.001"/>
+      </geometry>
+      <material name="grey"/>
+    </visual>
+    <collision>
+      <origin xyz="0 0 0" rpy="0 0 0"/>
+      <geometry>
+        <mesh filename="package://open_manipulator_p_description/meshes/link2.stl" scale="0.001 0.001 0.001"/>
+      </geometry>
+    </collision>
     <inertial>
       <origin xyz="0.00000 0.00080 0.03183" rpy="0 0 0"/>
@@ -66,17 +66,17 @@
   <!-- link 3 -->
   <link name="link3">
-    <collision>
-      <origin xyz="0 0 0" rpy="0 0 0"/>
-      <geometry>
-        <mesh filename="package://open_manipulator_p_description/meshes/link_3.stl" scale="0.001 0.001 0.001"/>
-      </geometry>
-    </collision>
-    <visual>
-      <origin xyz="0 0 0" rpy="0 0 0"/>
-      <geometry>
-        <mesh filename="package://open_manipulator_p_description/meshes/link_3.stl" scale="0.001 0.001 0.001"/>
-      </geometry>
-      <material name="grey"/>
-    </visual>
+    <visual>
+      <origin xyz="0 0 0" rpy="0 0 0"/>
+      <geometry>
+        <mesh filename="package://open_manipulator_p_description/meshes/link3.stl" scale="0.001 0.001 0.001"/>
+      </geometry>
+      <material name="grey"/>
+    </visual>
+    <collision>
+      <origin xyz="0 0 0" rpy="0 0 0"/>
+      <geometry>
+        <mesh filename="package://open_manipulator_p_description/meshes/link3.stl" scale="0.001 0.001 0.001"/>
+      </geometry>
+    </collision>
     <inertial>
       <origin xyz="0.01768 -0.06881 0.20524" rpy="0 0 0"/>
@@ -98,17 +98,17 @@
   <!-- link 4 -->
   <link name="link4">
-    <collision>
-      <origin xyz="0 0 0" rpy="0 0 0"/>
-      <geometry>
-        <mesh filename="package://open_manipulator_p_description/meshes/link_4.stl" scale="0.001 0.001 0.001"/>
-      </geometry>
-    </collision>
-    <visual>
-      <origin xyz="0 0 0" rpy="0 0 0"/>
-      <geometry>
-        <mesh filename="package://open_manipulator_p_description/meshes/link_4.stl" scale="0.001 0.001 0.001"/>
-      </geometry>
-      <material name="grey"/>
-    </visual>
+    <visual>
+      <origin xyz="0 0 0" rpy="0 0 0"/>
+      <geometry>
+        <mesh filename="package://open_manipulator_p_description/meshes/link4.stl" scale="0.001 0.001 0.001"/>
+      </geometry>
+      <material name="grey"/>
+    </visual>
+    <collision>
+      <origin xyz="0 0 0" rpy="0 0 0"/>
+      <geometry>
+        <mesh filename="package://open_manipulator_p_description/meshes/link4.stl" scale="0.001 0.001 0.001"/>
+      </geometry>
+    </collision>
     <inertial>
       <origin xyz="0.12475 -0.05716 0.02979" rpy="0 0 0"/>
@@ -130,17 +130,17 @@
   <!-- link 5 -->
   <link name="link5">
-    <collision>
-      <origin xyz="0 0 0" rpy="0 0 0"/>
-      <geometry>
-        <mesh filename="package://open_manipulator_p_description/meshes/link_5.stl" scale="0.001 0.001 0.001"/>
-      </geometry>
-    </collision>
-    <visual>
-      <origin xyz="0 0 0" rpy="0 0 0"/>
-      <geometry>
-        <mesh filename="package://open_manipulator_p_description/meshes/link_5.stl" scale="0.001 0.001 0.001"/>
-      </geometry>
-      <material name="grey"/>
-    </visual>
+    <visual>
+      <origin xyz="0 0 0" rpy="0 0 0"/>
+      <geometry>
+        <mesh filename="package://open_manipulator_p_description/meshes/link5.stl" scale="0.001 0.001 0.001"/>
+      </geometry>
+      <material name="grey"/>
+    </visual>
+    <collision>
+      <origin xyz="0 0 0" rpy="0 0 0"/>
+      <geometry>
+        <mesh filename="package://open_manipulator_p_description/meshes/link5.stl" scale="0.001 0.001 0.001"/>
+      </geometry>
+    </collision>
     <inertial>
       <origin xyz="0.05642 -0.00217 0.00002" rpy="0 0 0"/>
@@ -162,17 +162,17 @@
   <!-- link 6 -->
   <link name="link6">
-    <collision>
-      <origin xyz="0 0 0" rpy="0 0 0"/>
-      <geometry>
-        <mesh filename="package://open_manipulator_p_description/meshes/link_6.stl" scale="0.001 0.001 0.001"/>
-      </geometry>
-    </collision>
-    <visual>
-      <origin xyz="0 0 0" rpy="0 0 0"/>
-      <geometry>
-        <mesh filename="package://open_manipulator_p_description/meshes/link_6.stl" scale="0.001 0.001 0.001"/>
-      </geometry>
-      <material name="grey"/>
-    </visual>
+    <visual>
+      <origin xyz="0 0 0" rpy="0 0 0"/>
+      <geometry>
+        <mesh filename="package://open_manipulator_p_description/meshes/link6.stl" scale="0.001 0.001 0.001"/>
+      </geometry>
+      <material name="grey"/>
+    </visual>
+    <collision>
+      <origin xyz="0 0 0" rpy="0 0 0"/>
+      <geometry>
+        <mesh filename="package://open_manipulator_p_description/meshes/link6.stl" scale="0.001 0.001 0.001"/>
+      </geometry>
+    </collision>
     <inertial>
       <origin xyz="0.06831 -0.04457 0.00000" rpy="0 0 0"/>
@@ -222,17 +222,17 @@
   <!-- gripper main link -->
   <link name="gripper_main_link">
-    <collision>
+    <visual>
       <origin xyz="0 0 0" rpy="0 0 0" />
       <geometry>
         <mesh filename="package://open_manipulator_p_description/meshes/gripper_main_link.stl" scale="0.001 0.001 0.001"/>
       </geometry>
-    </collision>
-    <visual>
+      <material name="grey"/>
+    </visual>
+    <collision>
       <origin xyz="0 0 0" rpy="0 0 0" />
       <geometry>
         <mesh filename="package://open_manipulator_p_description/meshes/gripper_main_link.stl" scale="0.001 0.001 0.001"/>
       </geometry>
-      <material name="grey"/>
-    </visual>
+    </collision>
     <inertial>
       <origin xyz="0.0 0.0 0.0" rpy="0 0 0"/>
@@ -252,5 +252,5 @@
   <!-- gripper link -->
   <link name="gripper_link">
-    <collision>
+    <visual>
       <origin xyz="0 0 0" rpy="0 0 0" />
       <geometry>
@@ -258,6 +258,6 @@
       </geometry>
       <material name="grey"/>
-    </collision>
-    <visual>
+    </visual>
+    <collision>
       <origin xyz="0 0 0" rpy="0 0 0" />
       <geometry>
@@ -265,5 +265,5 @@
       </geometry>
       <material name="grey"/>
-    </visual>
+    </collision>
     <inertial>
       <origin xyz="0 0 0" rpy="0 0 0"/>
@@ -284,5 +284,5 @@
   <!-- gripper 1 link -->
   <link name="gripper_sub_link">
-    <collision>
+    <visual>
       <origin xyz="0 0 0" rpy="0 0 0" />
       <geometry>
@@ -290,6 +290,6 @@
       </geometry>
       <material name="grey"/>
-    </collision>
-    <visual>
+    </visual>
+    <collision>
       <origin xyz="0 0 0" rpy="0 0 0" />
       <geometry>
@@ -297,5 +297,5 @@
       </geometry>
       <material name="grey"/>
-    </visual>
+    </collision>
     <inertial>
       <origin xyz="0 0 0" rpy="0 0 0"/>

Commit message: update inertial info

File: open_manipulator_p_description/urdf/open_manipulator_p.urdf.xacro (robot description, xacro)
@@ -17,8 +17,9 @@
     </collision>
     <inertial>
-      <origin xyz="0.00023 0.00000 0.06223" rpy="0 0 0"/>
-      <mass value="0.85644"/>
-      <inertia ixx="1.0" ixy="0.0" ixz="0.0" iyy="1.0" iyz="0.0" izz="1.0" />
-      <!--<inertia ixx="0.00121064" ixy="0.0" ixz="0.00001100" iyy="0.00120886" iyz="0.0" izz="0.00038103" />-->
+      <origin xyz="0.0000000e+00 -1.7653633e-04 -1.0030209e-03" rpy="0 0 0"/>
+      <mass value="9.4360595e-01"/>
+      <inertia ixx="1.5684218e-03" ixy="0.0" ixz="0.0"
+               iyx="0.0" iyy="4.5498454e-04" iyz="1.7354214e-07"
+               izx="0.0" izy="1.7354214e-07" izz="1.5561515e-03" />
     </inertial>
   </link>
@@ -48,9 +49,9 @@
     </collision>
     <inertial>
-      <origin xyz="0.00000 0.00080 0.03183" rpy="0 0 0"/>
-      <!--<origin xyz="0.00000 -0.06820 -0.00117" rpy="0 0 0"/>-->
-      <mass value="0.94658"/>
-      <inertia ixx="1.0" ixy="0.0" ixz="0.0" iyy="1.0" iyz="0.0" izz="1.0" />
-      <!--<inertia ixx="0.00152547" ixy="0.0" ixz="0.0" iyy="0.00045954" iyz="-0.00001086" izz="0.00151740" />-->
+      <origin xyz="1.5751501e-02 -2.2073221e-04 1.9913687e-01" rpy="0 0 0"/>
+      <mass value="1.3825862e+00"/>
+      <inertia ixx="1.2803228e-02" ixy="-2.4795661e-05" ixz="-1.4109928e-03"
+               iyx="-2.4795661e-05" iyy="1.2037834e-02" iyz="1.4050354e-05"
+               izx="-1.4109928e-03" izy="1.4050354e-05" izz="2.2600348e-03" />
     </inertial>
   </link>
@@ -80,9 +81,9 @@
     </collision>
     <inertial>
-      <origin xyz="0.01768 -0.06881 0.20524" rpy="0 0 0"/>
-      <!--<origin xyz="-0.01232 -0.05731 -0.05876" rpy="0 0 0"/>-->
-      <mass value="1.30260"/>
-      <inertia ixx="1.0" ixy="0.0" ixz="0.0" iyy="1.0" iyz="0.0" izz="1.0" />
-      <!--<inertia ixx="0.01111021" ixy="0.00001331" ixz="-0.00134208" iyy="0.01046642" iyz="0.00016235" izz="0.00202081" />-->
+      <origin xyz="3.0352597e-04 4.1703880e-05 3.8074728e-01" rpy="0 0 0"/>
+      <mass value="1.2126965e+00"/>
+      <inertia ixx="4.0514666e-03" ixy="-9.7882420e-07" ixz="5.8582868e-05"
+               iyx="-9.7882420e-07" iyy="3.6839091e-03" iyz="1.5501165e-06"
+               izx="5.8582868e-05" izy="1.5501165e-06" izz="1.1420941e-03" />
     </inertial>
   </link>
@@ -112,9 +113,9 @@
     </collision>
     <inertial>
-      <origin xyz="0.12475 -0.05716 0.02979" rpy="0 0 0"/>
-      <!--<origin xyz="-0.07025 0.00034 -0.00021" rpy="0 0 0"/>-->
-      <mass value="1.15977"/>
-      <inertia ixx="1.0" ixy="0.0" ixz="0.0" iyy="1.0" iyz="0.0" izz="1.0" />
-      <!--<inertia ixx="0.00096726" ixy="0.00004383" ixz="-0.00002771" iyy="0.00318801" iyz="0.00000627" izz="0.00341484" />-->
+      <origin xyz="-2.1388493e-06 -2.2290515e-03 5.1387207e-01" rpy="0 0 0"/>
+      <mass value="4.6635550e-01"/>
+      <inertia ixx="4.2687885e-04" ixy="0.0000000e+00" ixz="0.0000000e+00"
+               iyx="0.0000000e+00" iyy="2.4774029e-04" iyz="3.5109263e-06"
+               izx="0.0000000e+00" izy="3.5109263e-06" izz="3.2985146e-04" />
     </inertial>
   </link>
@@ -144,9 +145,9 @@
     </collision>
     <inertial>
-      <origin xyz="0.05642 -0.00217 0.00002" rpy="0 0 0"/>
-      <!--<origin xyz="-0.00658 -0.04717 0.00002" rpy="0 0 0"/>-->
-      <mass value="0.44688"/>
-      <inertia ixx="1.0" ixy="0.0" ixz="0.0" iyy="1.0" iyz="0.0" izz="1.0" />
-      <!--<inertia ixx="0.00030285" ixy="0.00000761" ixz="0.00000031" iyy="0.00022339" iyz="-0.00000001" izz="0.00039766" />-->
+      <origin xyz="-2.1268822e-06 1.8039922e-04 5.9028250e-01" rpy="0 0 0"/>
+      <mass value="4.2561606e-01"/>
+      <inertia ixx="5.1431341e-04" ixy="0.0000000e+00" ixz="0.0000000e+00"
+               iyx="0.0000000e+00" iyy="4.2820999e-04" iyz="1.6136111e-06"
+               izx="0.0000000e+00" izy="1.6136111e-06" izz="2.1038697e-04" />
     </inertial>
   </link>
