Commit message: revise inertia

File: open_manipulator_p_description/urdf/open_manipulator_p.urdf.xacro (robot description, xacro)
@@ -19,7 +19,7 @@
       <origin xyz="0.0000000e+00 -1.7653633e-04 -1.0030209e-03" rpy="0 0 0"/>
       <mass value="9.4360595e-01"/>
-      <inertia ixx="1.5684218e-03" ixy="0.0" ixz="0.0"
-               iyx="0.0" iyy="4.5498454e-04" iyz="1.7354214e-07"
-               izx="0.0" izy="1.7354214e-07" izz="1.5561515e-03" />
+      <inertia ixx="1.0e-03" ixy="0.0" ixz="0.0"
+               iyx="0.0" iyy="1.0e-03" iyz="0.0"
+               izx="0.0" izy="0.0" izz="1.0e-03" />
     </inertial>
   </link>
@@ -49,9 +49,9 @@
     </collision>
     <inertial>
-      <origin xyz="1.5751501e-02 -2.2073221e-04 1.9913687e-01" rpy="0 0 0"/>
-      <mass value="1.3825862e+00"/>
-      <inertia ixx="1.2803228e-02" ixy="-2.4795661e-05" ixz="-1.4109928e-03"
-               iyx="-2.4795661e-05" iyy="1.2037834e-02" iyz="1.4050354e-05"
-               izx="-1.4109928e-03" izy="1.4050354e-05" izz="2.2600348e-03" />
+      <origin xyz="0.0000000e+00 -1.7653633e-04 -1.0030209e-03" rpy="0 0 0"/>
+      <mass value="9.4360595e-01"/>
+      <inertia ixx="1.5694005e-03" ixy="0.0" ixz="0.0"
+               iyx="0.0" iyy="4.5593385e-04" iyz="6.4581824e-09"
+               izx="0.0" izy="6.4581824e-09" izz="1.5561809e-03" />
     </inertial>
   </link>
@@ -81,9 +81,9 @@
     </collision>
     <inertial>
-      <origin xyz="3.0352597e-04 4.1703880e-05 3.8074728e-01" rpy="0 0 0"/>
-      <mass value="1.2126965e+00"/>
-      <inertia ixx="4.0514666e-03" ixy="-9.7882420e-07" ixz="5.8582868e-05"
-               iyx="-9.7882420e-07" iyy="3.6839091e-03" iyz="1.5501165e-06"
-               izx="5.8582868e-05" izy="1.5501165e-06" izz="1.1420941e-03" />
+      <origin xyz="1.5751501e-02 -2.2073221e-04 1.9913687e-01" rpy="0 0 0"/>
+      <mass value="1.3825862e+00"/>
+      <inertia ixx="6.7630430e-02" ixy="-1.9988597e-05" ixz="-5.7477571e-03"
+               iyx="-1.9988597e-05" iyy="6.7208001e-02" iyz="7.4823203e-05"
+               izx="-5.7477571e-03" izy="7.4823203e-05" izz="2.6031353e-03" />
     </inertial>
   </link>
@@ -113,9 +113,9 @@
     </collision>
     <inertial>
-      <origin xyz="-2.1388493e-06 -2.2290515e-03 5.1387207e-01" rpy="0 0 0"/>
-      <mass value="4.6635550e-01"/>
-      <inertia ixx="4.2687885e-04" ixy="0.0000000e+00" ixz="0.0000000e+00"
-               iyx="0.0000000e+00" iyy="2.4774029e-04" iyz="3.5109263e-06"
-               izx="0.0000000e+00" izy="3.5109263e-06" izz="3.2985146e-04" />
+      <origin xyz="3.0352597e-04 4.1703880e-05 3.8074728e-01" rpy="0 0 0"/>
+      <mass value="1.2126965e+00"/>
+      <inertia ixx="1.7985424e-01" ixy="-9.9417476e-07" ixz="-8.1564441e-05"
+               iyx="-9.9417476e-07" iyy="1.7948679e-01" iyz="-1.7705853e-05"
+               izx="-8.1564441e-05" izy="-1.7705853e-05" izz="1.1422079e-03" />
     </inertial>
   </link>
@@ -145,9 +145,9 @@
     </collision>
     <inertial>
-      <origin xyz="-2.1268822e-06 1.8039922e-04 5.9028250e-01" rpy="0 0 0"/>
-      <mass value="4.2561606e-01"/>
-      <inertia ixx="5.1431341e-04" ixy="0.0000000e+00" ixz="0.0000000e+00"
-               iyx="0.0000000e+00" iyy="4.2820999e-04" iyz="1.6136111e-06"
-               izx="0.0000000e+00" izy="1.6136111e-06" izz="2.1038697e-04" />
+      <origin xyz="-2.1388493e-06 -2.2290515e-03 5.1387207e-01" rpy="0 0 0"/>
+      <mass value="4.6635550e-01"/>
+      <inertia ixx="1.2357713e-01" ixy="-1.9465317e-09" ixz="5.1228604e-07"
+               iyx="-1.9465317e-09" iyy="1.2339567e-01" iyz="5.3769657e-04"
+               izx="5.1228604e-07" izy="5.3769657e-04" izz="3.3216863e-04" />
     </inertial>
   </link>
@@ -177,9 +177,9 @@
     </collision>
     <inertial>
-      <origin xyz="0.06831 -0.04457 0.00000" rpy="0 0 0"/>
-      <!--<origin xyz="-0.05469 0.00043 0.00000" rpy="0 0 0"/>-->
-      <mass value="0.43273"/>
-      <inertia ixx="1.0" ixy="0.0" ixz="0.0" iyy="1.0" iyz="0.0" izz="1.0" />
-      <!--<inertia ixx="0.00021512" ixy="0.00001009" ixz="0.00000000" iyy="0.00042827" iyz="0.00000000" izz="0.00051436" />-->
+      <origin xyz="-2.1268822e-06 1.8039922e-04 5.9028250e-01" rpy="0 0 0"/>
+      <mass value="4.2561606e-01"/>
+      <inertia ixx="1.4881319e-01" ixy="0.0000000e+00" ixz="5.3435266e-07"
+               iyx="0.0000000e+00" iyy="1.4872708e-01" iyz="-4.3708754e-05"
+               izx="5.3435266e-07" izy="-4.3708754e-05" izz="2.1040082e-04" />
     </inertial>
   </link>
@@ -211,6 +211,5 @@
       <origin xyz="0.00337 0.00000 0.00000" rpy="0 0 0"/>
       <mass value="0.01919"/>
-      <inertia ixx="1.0" ixy="0.0" ixz="0.0" iyy="1.0" iyz="0.0" izz="1.0" />
-      <!--<inertia ixx="0.00000938" ixy="0.0" ixz="0.0" iyy="0.00000338" iyz="0.0" izz="0.00000635" />-->
+      <inertia ixx="1.25e-4" ixy="0.0" ixz="0.0" iyy="1.25e-4" iyz="0.0" izz="1.25e-4" />
     </inertial>
   </link>
